File: vga_dvi_osvga.sch (KiCad schematic (older format))
At the start: 5 parts

Commit message: Add files via upload
Added Pull-up and pull-down resistors for JTAG and sysConfig connections.
Added pinheaders for FPGA-Configuration. (replacing edge-connector)
Combined the DVI+VGA and USB-C hierarchical sheets into one.
Assigned a dedicated sheet for the DAC.
Added 75 Ohm terminal-resistors to output of DAC.
Placed filtering-capacitors for DAC VAA.
Connected VGA ID-bits and DVI DDC together.
Parts:
- added J?: 2040210-1_NonStock, digikey-footprints:DisplayPort_2040210-1, symbol dk_USB-DVI-HDMI-Connectors:2040210-1_NonStock
- added USBC1: USB_C_Molex_201267-0005, Connector_USB:USB-C_Receptacle_2012670005, symbol LRJ-parts:USB_C_Molex_201267-0005
Connections:
- net labels added: +0V8, ABLUE, AGREEN, ARED, BLANK_DAC, BLUE0, BLUE1, BLUE2, BLUE3, BLUE4, BLUE5, BLUE6, BLUE7, CLK_DAC, DBLUE+, DBLUE-, DDC_CLK, DDC_DAT, GREEN0, GREEN1, GREEN2, GREEN3, GREEN4, GREEN5, GREEN6, GREEN7, RGB_ECP5, RST_DAC, SYNC_DAC, TMDS_CK+, TMDS_CK-
- net labels removed: 0.8V, BLAN, BLU0, BLU1, BLU2, BLU3, BLU4, BLU5, BLU6, BLU7, GRE0, GRE1, GRE2, GRE3, GRE4, GRE5, GRE6, GRE7, RGB_ECP5-85, SMPS_bus, SYN
- wire segments 180 -> 204
- no-connect marks 3 -> 0
Other:
- note added: "!"
- note added: "(2)"
- note added: "AUX CH +"
- note added: "AUX CH -"
- note added: "CONFIG1 (to gnd?)"
- note added: "CONFIG2 (to gnd?)"
- note added: "Config. Channels\n -role detect, et c"
- note added: "DP_PWR"
- note added: "GND"
- note added: "HOT PLUG (detect)"
- note added: "Hi-speed Data or \nDisPort alt mode"
- note added: "How to connect VGA DDC and DVI DDC??"
- note added: "ML_LANE 0 +"
- note added: "ML_LANE 0 -"
- note added: "ML_LANE 1 +"
- note added: "ML_LANE 1 -"
- note added: "ML_LANE 2 +"
- note added: "ML_LANE 2 -"
- note added: "ML_LANE 3 +"
- note added: "ML_LANE 3 -"
- note added: "P = +\nN = -"
- note added: "Return (for power)"
- note added: "Sideband \n- AUX for DisPort"
- note added: "USB 2.0 Data"
- note removed: "DDC Clock"
- note removed: "DDC Data"
- note removed: "Digital Blue + (2)"
- note removed: "Digital Blue - (2)"
- moved on the sheet: DAC1A, DAC1B, DAC1C, DAC1D, DAC1E, FPGA1C, FPGA1D
