File: DAC_60796DC7.sch (KiCad schematic (older format))
At the start: 15 parts

Commit message: Add files via upload
Connections:
- net M66EN_VT is gone; now on net SYNC_DAC: FPGA1.E20 (PR38A)
- net AUX+: now also FPGA1.L16 (PR50A/GR_PCLK3_0); no longer FPGA1.L20 (PR47A/PCLKT3_1)
- net AUX-: now also FPGA1.L17 (PR50B); no longer FPGA1.M20 (PR47B/PCLKC3_1)
- net BLANK_DAC: now also FPGA1.L18 (PR50C/GR_PCLK3_1); no longer FPGA1.M17 (PR53B)
- net BLUE2: now also FPGA1.T16 (PR77A); no longer FPGA1.U16 (PR92C/LRC_GPLL0T_IN)
- net SYNC_DAC: no longer FPGA1.N16 (PR53A)
- net TMDS_CK+: now also FPGA1.M20 (PR47B/PCLKC3_1); no longer FPGA1.L17 (PR50B)
- net TMDS_CK-: now also FPGA1.L20 (PR47A/PCLKT3_1); no longer FPGA1.L16 (PR50A/GR_PCLK3_0)
- net DBLUE-1: now reaches FPGA1.L19 (PR47C/PCLKT3_0)
- net DBLUE+1: now reaches FPGA1.M19 (PR47D/PCLKC3_0)
- net CS_DRAM: now reaches FPGA1.T17 (PR92D/LRC_GPLL0C_IN)
- net HPD_DVI: now reaches FPGA1.T20 (PR86C)
- new net DGREEN+1: FPGA1.N16 (PR53A)
- new net DGREEN-1: FPGA1.M17 (PR53B)
- new net ODT_DRAM: FPGA1.U16 (PR92C/LRC_GPLL0T_IN)
- no-connect marks 9 -> 3
Other:
- note added: "Control-signals \nfor the DRAM\nthat could not be\nfitted to banks\n2 and 3.\n<---"
- note added: "Resistor\nreference"
- moved on the sheet: FPGA1D
