File: svga-devboard.kicad_pcb (KiCad board)
At the start: 4 copper layers, 130 x 106.7 mm, 81 parts, among them J1 Bus_PCI_32bit_Universal_lrj, U1 SN74LVCH16T245DGGR, U2 SN74LVCH16T245DGGR, U3 SN74LVCH16T245DGGR, U4 SN74LVCH16T245DGGR

Commit message: Add files via upload
Parts:
- added C70: C1206C105K4RACTU, Capacitor_SMD:C_1206_3216Metric_Pad1.42x1.75mm_HandSolder, B.Cu at (130.9, 124.5)
- added C71: C1206C105K4RACTU, Capacitor_SMD:C_1206_3216Metric_Pad1.42x1.75mm_HandSolder, B.Cu at (135.0, 120.5)
- added C72: C1206C105K4RACTU, Capacitor_SMD:C_1206_3216Metric_Pad1.42x1.75mm_HandSolder, F.Cu at (158.0, 114.5)
- added C73: C1206C105K4RACTU, Capacitor_SMD:C_1206_3216Metric_Pad1.42x1.75mm_HandSolder, F.Cu at (166.5, 118.8)
- added C74: C1206C105K4RACTU, Capacitor_SMD:C_1206_3216Metric_Pad1.42x1.75mm_HandSolder, F.Cu at (175.2, 125.8)
- added C75: C1206C105K4RACTU, Capacitor_SMD:C_1206_3216Metric_Pad1.42x1.75mm_HandSolder, F.Cu at (181.2, 116.2)
- added C76: C1206C105K4RACTU, Capacitor_SMD:C_1206_3216Metric_Pad1.42x1.75mm_HandSolder, F.Cu at (149.8, 110.0)
- added C77: C1206C105K4RACTU, Capacitor_SMD:C_1206_3216Metric_Pad1.42x1.75mm_HandSolder, B.Cu at (151.2, 120.5)
- added C80: VJ1206Y104JXAAR, Capacitor_SMD:C_1206_3216Metric_Pad1.42x1.75mm_HandSolder, B.Cu at (130.9, 121.8)
- added C81: VJ1206Y104JXAAR, Capacitor_SMD:C_1206_3216Metric_Pad1.42x1.75mm_HandSolder, F.Cu at (137.5, 120.5)
- added C82: VJ1206Y104JXAAR, Capacitor_SMD:C_1206_3216Metric_Pad1.42x1.75mm_HandSolder, F.Cu at (158.0, 119.0)
- added C83: VJ1206Y104JXAAR, Capacitor_SMD:C_1206_3216Metric_Pad1.42x1.75mm_HandSolder, F.Cu at (158.8, 124.0)
- added C84: VJ1206Y104JXAAR, Capacitor_SMD:C_1206_3216Metric_Pad1.42x1.75mm_HandSolder, F.Cu at (182.0, 125.8)
- added C85: VJ1206Y104JXAAR, Capacitor_SMD:C_1206_3216Metric_Pad1.42x1.75mm_HandSolder, F.Cu at (181.5, 121.0)
- added C86: VJ1206Y104JXAAR, Capacitor_SMD:C_1206_3216Metric_Pad1.42x1.75mm_HandSolder, F.Cu at (149.8, 114.2)
- added C87: VJ1206Y104JXAAR, Capacitor_SMD:C_1206_3216Metric_Pad1.42x1.75mm_HandSolder, B.Cu at (148.8, 120.5)
- added C90: VJ1206Y104JXAAR, Capacitor_SMD:C_1206_3216Metric_Pad1.42x1.75mm_HandSolder, F.Cu at (134.0, 113.0)
- added C91: VJ1206Y104JXAAR, Capacitor_SMD:C_1206_3216Metric_Pad1.42x1.75mm_HandSolder, F.Cu at (128.8, 113.0)
- added C92: VJ1206Y104JXAAR, Capacitor_SMD:C_1206_3216Metric_Pad1.42x1.75mm_HandSolder, F.Cu at (166.2, 114.2)
- added C93: VJ1206Y104JXAAR, Capacitor_SMD:C_1206_3216Metric_Pad1.42x1.75mm_HandSolder, F.Cu at (166.8, 124.0)
- added C94: VJ1206Y104JXAAR, Capacitor_SMD:C_1206_3216Metric_Pad1.42x1.75mm_HandSolder, F.Cu at (174.6, 120.6)
- added C95: VJ1206Y104JXAAR, Capacitor_SMD:C_1206_3216Metric_Pad1.42x1.75mm_HandSolder, F.Cu at (174.7, 116.0)
- added C96: VJ1206Y104JXAAR, Capacitor_SMD:C_1206_3216Metric_Pad1.42x1.75mm_HandSolder, F.Cu at (143.8, 109.8)
- added C97: VJ1206Y104JXAAR, Capacitor_SMD:C_1206_3216Metric_Pad1.42x1.75mm_HandSolder, F.Cu at (143.8, 114.5)
- added RZQ1: ERJ-8ENF2400V, Resistor_SMD:R_Panasonic_1206_3216Metric_ERJ8EN_HandSolder, B.Cu at (153.0, 87.0)
- moved U1 4.00 mm to (131.4, 120.2)
- moved U2 4.00 mm to (162.1, 120.2)
- moved U3 4.00 mm to (177.9, 120.2)
- moved U4 4.00 mm to (146.5, 120.2)
Connections:
- net Net-(DVI1-Pad10) renamed /VGA + DVI + USBC/DGREEN+1
- net Net-(DVI1-Pad16) renamed /VGA + DVI + USBC/HPD_DVI
- net Net-(DVI1-Pad17) renamed /VGA + DVI + USBC/DBLUE-1
- net Net-(DVI1-Pad18) renamed /VGA + DVI + USBC/DBLUE+1
- net Net-(DVI1-Pad9) renamed /VGA + DVI + USBC/DGREEN-1
- net Net-(FPGA1-PadE15) renamed /FPGA GPU/M66EN_VT
- net Net-(FPGA1-PadL19) renamed /DAC/DBLUE-1
- net Net-(FPGA1-PadM19) renamed /DAC/DBLUE+1
- net Net-(FPGA1-PadT17) renamed /DAC/CS_DRAM
- net Net-(FPGA1-PadT20) renamed /DAC/HPD_DVI
- net Net-(LPDDR3-PadJ8) renamed /DRAM/ODT_DRAM
- net Net-(LPDDR3-PadL3) renamed /DRAM/CS_DRAM
- DVI1 pad C2: /VGA + DVI + USBC/ABLUE -> /VGA + DVI + USBC/AGREEN
- DVI1 pad C3: /VGA + DVI + USBC/AGREEN -> /VGA + DVI + USBC/ABLUE
- FPGA1 pad E20: /DAC/M66EN_VT -> /DAC/SYNC_DAC
- FPGA1 pad L16: /DAC/TMDS_CK- -> /DAC/AUX+
- FPGA1 pad L17: /DAC/TMDS_CK+ -> /DAC/AUX-
- FPGA1 pad L18: Net-(FPGA1-PadL18) -> /DAC/BLANK_DAC
- FPGA1 pad L20: /DAC/AUX+ -> /DAC/TMDS_CK-
- FPGA1 pad M17: /DAC/BLANK_DAC -> /DAC/DGREEN-1
- FPGA1 pad M20: /DAC/AUX- -> /DAC/TMDS_CK+
- FPGA1 pad N16: /DAC/SYNC_DAC -> /DAC/DGREEN+1
- FPGA1 pad T16: Net-(FPGA1-PadT16) -> /DAC/BLUE2
- FPGA1 pad U16: /DAC/BLUE2 -> /DAC/ODT_DRAM
- J1 pad B57: Net-(J1-PadB57) -> GND
- LPDDR3 pad J3: /DRAM/CK_c_DRAM -> /DRAM/CK_t_DRAM
- U1 pad 18: +5V -> +1V2
- U1 pad 31: +3V3 -> +5V
- U1 pad 7: +5V -> +1V2
- U2 pad 18: +5V -> +1V2
- U2 pad 31: +3V3 -> +5V
- U2 pad 7: +5V -> +1V2
- U3 pad 18: +5V -> +1V2
- U3 pad 31: +3V3 -> +5V
- U3 pad 7: +5V -> +1V2
- U4 pad 18: +5V -> +1V2
- U4 pad 31: +3V3 -> +5V
- U4 pad 7: +5V -> +1V2
Routing:
- net +5V: track 293.9 -> 176.9 mm, vias 16 -> 12
- net GND: track 851.5 -> 745.7 mm, vias 107 -> 104
- net +1V2: track 0.00 -> 81.2 mm, vias 0 -> 6
- net /Signal Voltage-level translation/RST_VT: track 28.5 -> 0.00 mm
- net +3V3: track 152.3 -> 127.0 mm, vias 18 -> 13
- net /Signal Voltage-level translation/CLK_VT: track 22.1 -> 0.00 mm
- net /PCI/PCI_AD28: track 20.5 -> 0.00 mm, vias 1 -> 0
- net /Signal Voltage-level translation/REQ_VT: track 18.0 -> 0.00 mm
- net /PCI/PCI_TRST: track 17.7 -> 0.00 mm, vias 1 -> 0
- net /PCI/PCI_AD29: track 17.5 -> 0.00 mm
- net /PCI/PCI_AD31: track 16.8 -> 0.00 mm
- net /Signal Voltage-level translation/PME_VT: track 16.7 -> 0.00 mm
- net /PCI/PCI_AD30: track 16.4 -> 0.00 mm, vias 1 -> 0
- net /PCI/PCI_PME: track 15.9 -> 0.00 mm, vias 1 -> 0
- net /Signal Voltage-level translation/AD30_VT: track 15.6 -> 0.00 mm
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