File: Hardware/svga-devboard/VoltTranslate_osvga.kicad_sch (KiCad schematic)
At the start: 29 parts, among them U2 SN74LVCH16T245DGGR, U3 SN74LVCH16T245DGGR, U4 SN74LVCH16T245DGGR, U5 SN74LVCH16T245DGGR

Commit message: Disconnected the DVI-connectors from each other, so that they do go over the intended flat-cable to the daughter-board instead.
Parts:
- C10, C11, C12, C13, C16, C17, C18, C19, C22, C23, C24, C25, C4, C5, C6, C7: value VJ1206Y104JXAAR -> C_CC0805JPX7R9BB104; footprint Capacitor_SMD:C_1206_3216Metric -> Capacitor_SMD:C_0805_2012Metric; symbol LRJ-parts:C_VJ1206Y104JXAAR -> LRJ-parts:C_CC0805JPX7R9BB104; Capacitance (none) -> 0.1uF; Capacity 0.1uF -> (none); MPN VJ1206Y104JXAAR -> CC0805JPX7R9BB104; Manufacturer Vishay / Vitramon -> Yageo; Mounting type (none) -> SMD; Status (none) -> Active; Temperature Coefficient  (none) -> X7R
- C14, C15, C2, C20, C21, C3, C8, C9: value C_C1206C105K4 -> C_CL21B105KBFNNNF; footprint Capacitor_SMD:C_1206_3216Metric_Pad1.33x1.80mm_HandSolder -> Capacitor_SMD:C_0805_2012Metric_Pad1.18x1.45mm_HandSolder; symbol LRJ-parts:C_C1206C105K4 -> LRJ-parts:C_CL21B105KBFNNNF; Capacitance (none) -> 1 µF; Capacity 1uF -> (none); MPN C1206C105K4RACTU -> CL21B105KBFNNNF; Manufacturer KEMET -> Samsung Electro-Mechanics; Voltage rating (none) -> 50V
Other:
- note added: "The VT_ -moniker denotes that the signal has been voltage-Translated, from 5V/3.3V, into a lower voltage-level that is more compatible with current technologies."
- note removed: "The VT_ -moniker denotes that the signal have been Voltage-Translated, from 5V/3.3V, into a lower voltage-level that is more compatible with current technologies."
- moved on the sheet: R24, U2A, U2B, U3A, U3B, U4A, U4B, U5A, U5B
