File: Hardware/svga-devboard/ecp5-85-fpga.kicad_sch (KiCad schematic)
At the start: 1 part

Commit message: Disconnected the DVI-connectors from each other, so that they do go over the intended flat-cable to the daughter-board instead.
Parts:
- added unit 7 of FPGA1
- added Flash1: ISSI_IS25WP128F-JBLE, Footprints:SOIC-8_5.28x5.28mm_P1.27mm, symbol LRJ-parts:ISSI_IS25WP128F-JBLE
- added J2: Wurth_WR-BHD_61201021721, LRJ:Wuerth_WR-BHD_61201021721_2x05_P2.54mm_Horizontal, symbol LRJ-parts:Wurth_WR-BHD_61201021721
- added JTAG1: Conn_NREC004, Connector_PinHeader_2.54mm:PinHeader_1x04_P2.54mm_Vertical_SMD_Pin1Right, symbol LRJ-parts:Conn_NREC004
- added R1, R2, R3, R37, R4, R5, R6, R7, R8: R_ERJ-P06F1001V, Resistor_SMD:R_0805_2012Metric_Pad1.20x1.40mm_HandSolder, symbol LRJ-parts:R_ERJ-P06F1001V
Connections:
- net DIR_21: now also FPGA1.T3 (PB18A/WRITEN); no longer FPGA1.E3 (PL20B)
- net DIR_32: now also FPGA1.U2 (PB13B/CS1N); no longer FPGA1.A2 (PL35A)
- net OE_21: now also FPGA1.R1 (PB4A/D7/IO7); no longer FPGA1.F4 (PL20A)
- net OE_32: now also FPGA1.T2 (PB13A/SN/CSN); no longer FPGA1.B1 (PL35B)
- new net +1V8: Flash1.8 (VCC)
- new net +2V5: R1.2, R2.2, R3.2, R37.2, R4.2, R5.2, R6.2
- new net CFG_0: FPGA1.U4 (CFG_0), R8.1
- new net CFG_1: FPGA1.T4 (CFG_1), R6.1
- new net CFG_2: FPGA1.R4 (CFG_2), R7.1
- new net CSSPIN_FPGA: FPGA1.R2 (PB15A/HOLDN/DI/BUSY/CSSPIN/CEN), Flash1.1 (CE#), J2.7, R37.1
- new net DOUT_FPGA: FPGA1.R3 (PB15B/DOUT/CSON), J2.5
- new net DUSB_1+: FPGA1.B1 (PL35B)
- new net DUSB_1-: FPGA1.A2 (PL35A)
- new net DUSB_2+: FPGA1.E3 (PL20B)
- new net DUSB_2-: FPGA1.F4 (PL20A)
- new net GND: Flash1.4 (GND), J2.9, R7.2, R8.2
- new net INIT_FPGA: FPGA1.V3 (INITN), J2.3
- new net IO2_FPGA: FPGA1.Y2 (PB9B/D2/IO2), Flash1.3 (WP#/IO2), J2.6, R4.1
- new net IO3_FPGA: FPGA1.W1 (PB9A/D3/IO3), Flash1.7 (RST#/IO3), J2.8, R5.1
- new net MCLK_FPGA: FPGA1.U3 (CCLK/MCLK/SCK), Flash1.6 (SCK), J2.10, R1.1
- new net MISO_FPGA: FPGA1.U1 (PB6A/D5/MISO2/IO5), Flash1.2 (SO/IO1), J2.4, R3.1
- new net MOSI_FPGA: FPGA1.V1 (PB6B/D4/MOSI2/IO4), Flash1.5 (SI/IO0), J2.2, R2.1
- new net PROG_FPGA: FPGA1.W3 (PROGRAMN), J2.1
- new net RAM_PG2: FPGA1.W2 (PB11B/D0/MOSI/IO0)
- new net TCK_FPGA: FPGA1.T5 (TCK), JTAG1.4 (Pin_4)
- new net TDI_FPGA: FPGA1.R5 (TDI), JTAG1.3 (Pin_3)
- new net TDO_FPGA: FPGA1.V4 (TDO), JTAG1.2 (Pin_2)
- new net TMS_FPGA: FPGA1.U5 (TMS), JTAG1.1 (Pin_1)
- no-connect marks 0 -> 3
Other:
- note added: "0"
- note added: "1"
- note added: "<- USB 2.0"
- note added: "CE# enables operation of flash chip. Set to High (+V) when progr. w. JTAG."
- note added: "CONFIGURATION"
- note added: "DIR ->"
- note added: "Pull-ups for QUAD Master SPI"
- note added: "VIDEO OUTPUT DIGITAL"
- moved on the sheet: FPGA1E
