File: Hardware/svga-devboard/jtag_osvga.kicad_sch (KiCad schematic)
At the start: 13 parts, among them J2 Wurth_WR-BHD_61201021721

Commit message: Disconnected the DVI-connectors from each other, so that they do go over the intended flat-cable to the daughter-board instead.
Parts:
- removed FPGA1: LFE5U-85F-8BG381, LRJ:Lattice_caBGA-381_17.0x17.0_Layout18x18_P0.8_Ball0.4_Pad0.4mm_LRJ, symbol LRJ-parts:LFE5U-85F-8BG381
- removed Flash1: ISSI_IS25WP128F-JBLE, Footprints:SOIC-8_5.28x5.28mm_P1.27mm, symbol LRJ-parts:ISSI_IS25WP128F-JBLE
- removed J2: Wurth_WR-BHD_61201021721, LRJ:Wuerth_WR-BHD_61201021721_2x05_P2.54mm_Horizontal, symbol LRJ-parts:Wurth_WR-BHD_61201021721
- removed JTAG1: Conn_NREC004, Connector_PinHeader_2.54mm:PinHeader_1x04_P2.54mm_Vertical_SMD_Pin1Right, symbol LRJ-parts:Conn_NREC004
- removed R1, R2, R3, R37, R4, R5, R6, R7, R8: R_ERJ-P06F1001V, Resistor_SMD:R_0805_2012Metric_Pad1.20x1.40mm_HandSolder, symbol LRJ-parts:R_ERJ-P06F1001V
Connections:
- no-connect marks 7 -> 0
Other:
- note removed: "0"
- note removed: "1"
- note removed: "CE# enables operation of flash chip. Set to High (+V) when progr. w. JTAG."
- note removed: "Pull-ups for QUAD Master SPI"
